File: hardware/328p.kicad_sch (KiCad schematic)
At the start: 12 parts, among them J3 AVR-ISP-6, SW2 SW_Push, U2 ATmega328P-A, Y1 8MHz

Commit message: Infinite schematic/PCB changes
Parts:
- removed C8: 10uF, Capacitor_SMD:C_0805_2012Metric, symbol Device:C
Connections:
- net VCC renamed MCU_VCC
Other:
- note removed: "0.1 uF: 603 10 uF: 805"
- moved on the sheet: C4

Commit message: Keep hacking
Parts:
- removed C10, C9: 22pF, Capacitor_SMD:C_0603_1608Metric, symbol Device:C_Small
- removed Y1: 8MHz, Crystal:Crystal_SMD_2012-2Pin_2.0x1.2mm, symbol Device:Crystal
- added Y2: Resonator, Crystal:Resonator_SMD_Murata_CSTxExxV-3Pin_3.0x1.1mm, symbol Device:Resonator
- renumbered C11 to C1, J3 to J1, R5 to R1, SW2 to SW1, U2 to U1
Connections:
- net GND: now also Y2.2
- net XTAL1: now also Y2.3
- net XTAL2: now also Y2.1

Commit message: Further PCB tweaks
Parts:
- added R16: 0, Resistor_SMD:R_1206_3216Metric_Pad1.30x1.75mm_HandSolder, symbol Device:R
Connections:
- net MCU_VCC: now also R16.1, R16.2
