File: hardware/coffee-scales.kicad_pcb (KiCad board)
At the start: 2 copper layers, 121.9 x 50.8 mm, 41 parts, among them J1 AVR-ISP-6, J2 Conn_01x05, Q1 MMBT4403, SW1 SW_Push, SW2 SW_Push, U1 ATmega328P-A, Y2 Resonator

Commit message: Further PCB tweaks
Parts:
- removed TP2: TestPoint, TestPoint:TestPoint_THTPad_D1.0mm_Drill0.5mm
- added C17: 4.7uF, Capacitor_SMD:C_0805_2012Metric, F.Cu at (43.2, 119.6)
- added C18: 10uF, Capacitor_SMD:C_0805_2012Metric, F.Cu at (54.9, 107.3)
- added C2: 1uF, Capacitor_SMD:C_0603_1608Metric, F.Cu at (53.2, 104.8)
- added C3: 1uF, Capacitor_SMD:C_0603_1608Metric, F.Cu at (66.7, 114.3)
- added D2: LED, LED_SMD:LED_0805_2012Metric, F.Cu at (52.1, 122.6)
- added J3: Conn_01x02_Pin, Connector_JST:JST_PH_S2B-PH-SM4-TB_1x02-1MP_P2.00mm_Horizontal, F.Cu at (55.1, 98.8)
- added J4: USB_C_Receptacle_PowerOnly_6P, Connector_USB:USB_C_Receptacle_GCT_USB4125-xx-x-0190_6P_TopMnt_Horizontal, F.Cu at (36.8, 120.5)
- added J5: Conn_01x01, TestPoint:TestPoint_Pad_D1.5mm, F.Cu at (146.1, 125.7)
- added J6: Conn_01x01, TestPoint:TestPoint_Pad_D1.5mm, F.Cu at (138.4, 125.7)
- added J7: Conn_01x01, TestPoint:TestPoint_Pad_D1.5mm, F.Cu at (135.9, 125.7)
- added J8: Conn_01x01, TestPoint:TestPoint_Pad_D1.5mm, F.Cu at (143.5, 125.7)
- added R11: 10k, Resistor_SMD:R_0603_1608Metric, F.Cu at (59.1, 114.3)
- added R12: 470, Resistor_SMD:R_0603_1608Metric, F.Cu at (54.0, 119.4)
- added R13: 2k, LED_SMD:LED_0603_1608Metric, F.Cu at (52.1, 119.4)
- added R14: 5.1k, Resistor_SMD:R_0603_1608Metric, F.Cu at (44.0, 124.3)
- added R15: 5.1k, Resistor_SMD:R_0603_1608Metric, F.Cu at (44.0, 122.4)
- added U7: TPS78233DDC, Package_TO_SOT_SMD:SOT-23-5, F.Cu at (62.7, 114.3)
- added U8: MCP73831-2-OT, Package_TO_SOT_SMD:SOT-23-5, F.Cu at (48.9, 117.5)
- J2: value Conn_01x05 -> Conn_01x01; footprint Connector_PinSocket_2.54mm:PinSocket_1x05_P2.54mm_Horizontal -> TestPoint:TestPoint_Pad_D1.5mm
- moved J2 11.7 mm to (141.0, 125.7), turned to 0 degrees
- moved C9 10.2 mm to (143.6, 129.5)
- moved C10 9.83 mm to (144.3, 132.1)
- moved TP1 2.84 mm to (115.6, 139.7)
- moved L1 1.91 mm to (135.3, 136.5)
- moved R1 1.65 mm to (59.1, 132.9), turned to 90 degrees
- moved Y2 0.64 mm to (71.8, 129.5)
- moved NT1 0.50 mm to (116.1, 138.4)
Connections:
- net GND renamed -BATT
- C10 pad 2: HX_GNDA -> GNDA
- C5 pad 2: HX_GNDA -> GNDA
- C6 pad 1: HX_GNDA -> GNDA
- C8 pad 2: HX_GNDA -> GNDA
- C9 pad 2: HX_GNDA -> GNDA
- NT1 pad 1: HX_GNDA -> GNDA
- R5 pad 2: HX_GNDA -> GNDA
- U2 pad 10: HX_GNDA -> GNDA
- U2 pad 14: HX_GNDA -> GNDA
- U2 pad 15: HX_GNDA -> GNDA
- U2 pad 5: HX_GNDA -> GNDA
- U2 pad 9: HX_GNDA -> GNDA
Routing:
- net +BATT: track 0.00 -> 29.0 mm
- net VCC: track 205.3 -> 181.4 mm, vias 9 -> 8
- net VUSB: track 0.00 -> 19.1 mm
- net /HX711/A-: track 17.3 -> 5.47 mm
- net /HX711/A+: track 11.9 -> 2.14 mm
- net Net-(U8-STAT): track 0.00 -> 5.68 mm
- net Net-(J4-CC2): track 0.00 -> 4.92 mm
- net Net-(J4-CC1): track 0.00 -> 4.27 mm
- net /HX711/E+: track 20.8 -> 16.6 mm
- net -BATT: track 9.10 -> 12.5 mm, vias 2 -> 104
- net Net-(D2-K): track 0.00 -> 2.75 mm
- net Net-(U7-EN): track 0.00 -> 2.59 mm
- net Net-(U8-PROG): track 0.00 -> 2.23 mm
- net HX_GNDA: track 2.04 -> 0.00 mm, vias 3 -> 0
- net /328P/XTAL2: track 3.58 -> 4.96 mm
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- added copper zone on B.Cu, net GNDA
- added copper zone on F.Cu, net GNDA
- removed copper zone on B.Cu, net HX_GNDA
- removed copper zone on F.Cu, net HX_GNDA
Other:
- board size 121.9 x 50.8 mm -> 121.9 x 78.7 mm
- board text added: "Press to turn on or tare Long press to turn off"
- board text added: "mortenfyhn/coffee-scales Rev 2"
- board text removed: "Decoupling"
- board text removed: "Reset stuff"
- board text removed: "mortenfyhn/coffee-scales Rev2"
- board text removed: "·Press to turn on ·Press to tare ·Long press to turn off"
