File: hardware/coffee-scales.kicad_sch (KiCad schematic)
At the start: 5 parts, among them J2 Conn_01x05, SW1 SW_Push, U3 4DIGIT_7SEG, U4 4DIGIT_7SEG

Commit message: Infinite schematic/PCB changes
Parts:
- removed U3, U4: 4DIGIT_7SEG, CoffeeLib:4DIGIT_7SEG, symbol CoffeeLib:4DIGIT_7SEG
Connections:
- no-connect marks 6 -> 0
Other:
- added sheet Gram display (display.kicad_sch)
- added sheet Time display (display.kicad_sch)
- sheet 328P ports: added MCU_VCC; removed none
- note removed: "Scale display"
- note removed: "Timer display"
- moved on the sheet: J2, NT1, SW1

Commit message: Keep hacking
Parts:
- added TP1, TP2: TestPoint, TestPoint:TestPoint_THTPad_D1.0mm_Drill0.5mm, symbol Connector:TestPoint
- renumbered SW1 to SW2
Connections:
- net GND: now also TP1.1
- net HX711/HX_GNDA: now also TP2.1
Other:
- moved on the sheet: J2, NT1

Commit message: Further PCB tweaks
Parts:
- removed J2: Conn_01x05, Connector_PinSocket_2.54mm:PinSocket_1x05_P2.54mm_Horizontal, symbol Connector_Generic:Conn_01x05
- removed TP2: TestPoint, TestPoint:TestPoint_THTPad_D1.0mm_Drill0.5mm, symbol Connector:TestPoint
- added C17: 4.7uF, Capacitor_SMD:C_0805_2012Metric, symbol Device:C_Small
- added C18: 10uF, Capacitor_SMD:C_0805_2012Metric, symbol Device:C_Small
- added C2, C3: 1uF, Capacitor_SMD:C_0603_1608Metric, symbol Device:C_Small
- added D2: LED, LED_SMD:LED_0805_2012Metric, symbol Device:LED
- added J2, J5, J6, J7, J8: Conn_01x01, TestPoint:TestPoint_Pad_D1.5mm, symbol Connector_Generic:Conn_01x01
- added J3: Conn_01x02_Pin, Connector_JST:JST_PH_S2B-PH-SM4-TB_1x02-1MP_P2.00mm_Horizontal, symbol Connector:Conn_01x02_Pin
- added J4: USB_C_Receptacle_PowerOnly_6P, Connector_USB:USB_C_Receptacle_GCT_USB4125-xx-x-0190_6P_TopMnt_Horizontal, symbol Connector:USB_C_Receptacle_PowerOnly_6P
- added R11: 10k, Resistor_SMD:R_0603_1608Metric, symbol Device:R
- added R12: 470, Resistor_SMD:R_0603_1608Metric, symbol Device:R
- added R13: 2k, LED_SMD:LED_0603_1608Metric, symbol Device:R
- added R14, R15: 5.1k, Resistor_SMD:R_0603_1608Metric, symbol Device:R
- added U7: TPS78233DDC, Package_TO_SOT_SMD:SOT-23-5, symbol Regulator_Linear:TPS78233DDC
- added U8: MCP73831-2-OT, Package_TO_SOT_SMD:SOT-23-5, symbol Battery_Management:MCP73831-2-OT
Connections:
- net HX711/A+: now also J7.1 (Pin_1)
- net HX711/A-: now also J6.1 (Pin_1)
- net HX711/E+: now also J2.1 (Pin_1)
- net HX711/E-: now also J5.1 (Pin_1)
- net HX711/SHLD: now also J8.1 (Pin_1)
- net VCC: now also C3.1, U7.5 (OUT)
- net GND renamed -BATT
- net -BATT: now also C17.2, C18.2, C2.2, C3.2, J3.1 (Pin_1), J4.A12 (GND), J4.B12 (GND), J4.S1 (SHIELD), R13.2, R14.2, R15.2, U7.2 (GND), U7.4 (GND), U8.2 (V_{SS})
- net HX711/HX_GNDA renamed HX711/GNDA
- new net: R12.1, U8.1 (STAT)
- new net: R13.1, U8.5 (PROG)
- new net: D2.1 (K), R12.2
- new net: J4.A5 (CC1), R15.1
- new net: J4.B5 (CC2), R14.1
- new net: R11.2, U7.3 (EN)
- new net +BATT: C18.1, C2.1, J3.2 (Pin_2), R11.1, U7.1 (IN), U8.3 (V_{BAT})
- new net VUSB: C17.1, D2.2 (A), J4.A9 (VBUS), J4.B9 (VBUS), U8.4 (V_{DD})
Other:
- sheet HX711 ports: added DAT, GNDA, SCK, VCC, VDD; removed HX_DAT, HX_GNDA, HX_SCK, HX_VCC, HX_VDD
- moved on the sheet: NT1, TP1
