File: hardware/display.kicad_sch (KiCad schematic)
At the start: 7 parts

Commit message: Keep hacking
Parts:
- U3: renamed from U1; footprint Package_SO:SOP-20_7.5x12.8mm_P1.27mm -> CoffeeLib:SOP-20_7.5x12.8mm_P1.27mm_3d
- renumbered C15 to C11, C16 to C12, C19 to C13, R9 to R7, U7 to U4
Changed lines of the file:
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@@
 		(on_board yes)
 		(dnp no)
-		(property "Reference" "U7"
+		(property "Reference" "U4"
 			(at 207.01 92.202 0)
 			(effects
@@
 			(project "coffee-scales"
 				(path "/2c28a4aa-0841-4fd8-a9c6-3f977db869be/031c2cff-942d-4852-b066-d842581777eb"
-					(reference "U7")
+					(reference "U4")
 					(unit 1)
 				)
@@
 		(dnp no)
 		(fields_autoplaced yes)
-		(property "Reference" "R9"
+		(property "Reference" "R7"
 			(at 127 66.0399 0)
 			(effects
@@
 			(project "coffee-scales"
 				(path "/2c28a4aa-0841-4fd8-a9c6-3f977db869be/031c2cff-942d-4852-b066-d842581777eb"
+					(reference "R7")
+					(unit 1)
+				)
+				(path "/2c28a4aa-0841-4fd8-a9c6-3f977db869be/ac5a0b65-b34e-4c1b-aa94-9c346f583af7"
 					(reference "R9")
-					(unit 1)
-				)
-				(path "/2c28a4aa-0841-4fd8-a9c6-3f977db869be/ac5a0b65-b34e-4c1b-aa94-9c346f583af7"
-					(reference "R7")
 					(unit 1)
 				)
@@
 		(dnp no)
 		(fields_autoplaced yes)
-		(property "Reference" "C16"
+		(property "Reference" "C12"
 			(at 144.78 72.3962 0)
 			(effects
@@
 			(project "coffee-scales"
 				(path "/2c28a4aa-0841-4fd8-a9c6-3f977db869be/031c2cff-942d-4852-b066-d842581777eb"
-					(reference "C16")
-					(unit 1)
-				)
-				(path "/2c28a4aa-0841-4fd8-a9c6-3f977db869be/ac5a0b65-b34e-4c1b-aa94-9c346f583af7"
-					(reference "C17")
+					(reference "C12")
+					(unit 1)
+				)
+				(path "/2c28a4aa-0841-4fd8-a9c6-3f977db869be/ac5a0b65-b34e-4c1b-aa94-9c346f583af7"
+					(reference "C14")
 					(unit 1)
 				)
@@
 		(dnp no)
 		(fields_autoplaced yes)
-		(property "Reference" "C15"
+		(property "Reference" "C11"
 			(at 127 72.3962 0)
 			(effects
@@
 			(project "coffee-scales"
 				(path "/2c28a4aa-0841-4fd8-a9c6-3f977db869be/031c2cff-942d-4852-b066-d842581777eb"
+					(reference "C11")
+					(unit 1)
+				)
+				(path "/2c28a4aa-0841-4fd8-a9c6-3f977db869be/ac5a0b65-b34e-4c1b-aa94-9c346f583af7"
 					(reference "C15")
-					(unit 1)
-				)
-				(path "/2c28a4aa-0841-4fd8-a9c6-3f977db869be/ac5a0b65-b34e-4c1b-aa94-9c346f583af7"
-					(reference "C13")
 					(unit 1)
 				)
@@
 		(on_board yes)
 		(dnp no)
-		(property "Reference" "U1"
+		(property "Reference" "U3"
 			(at 160.02 92.202 0)
 			(effects
@@
 			)
 		)
-		(property "Footprint" "Package_SO:SOP-20_7.5x12.8mm_P1.27mm"
+		(property "Footprint" "CoffeeLib:SOP-20_7.5x12.8mm_P1.27mm_3d"
 			(at 160.02 107.95 0)
 			(effects
@@
 			(project "coffee-scales"
 				(path "/2c28a4aa-0841-4fd8-a9c6-3f977db869be/031c2cff-942d-4852-b066-d842581777eb"
-					(reference "U1")
-					(unit 1)
-				)
-				(path "/2c28a4aa-0841-4fd8-a9c6-3f977db869be/ac5a0b65-b34e-4c1b-aa94-9c346f583af7"
 					(reference "U3")
+					(unit 1)
+				)
+				(path "/2c28a4aa-0841-4fd8-a9c6-3f977db869be/ac5a0b65-b34e-4c1b-aa94-9c346f583af7"
+					(reference "U5")
 					(unit 1)
 				)
@@
 		(dnp no)
 		(fields_autoplaced yes)
-		(property "Reference" "C19"
+		(property "Reference" "C13"
 			(at 163.83 67.3162 0)
 			(effects
@@
 			(project "coffee-scales"
 				(path "/2c28a4aa-0841-4fd8-a9c6-3f977db869be/031c2cff-942d-4852-b066-d842581777eb"
-					(reference "C19")
-					(unit 1)
-				)
-				(path "/2c28a4aa-0841-4fd8-a9c6-3f977db869be/ac5a0b65-b34e-4c1b-aa94-9c346f583af7"
-					(reference "C18")
-					(unit 1)
-				)
+					(reference "C13")
+					(unit 1)
+				)
+				(path "/2c28a4aa-0841-4fd8-a9c6-3f977db869be/ac5a0b65-b34e-4c1b-aa94-9c346f583af7"
+					(reference "C16")
+					(unit 1)
+				)
