File: hardware/hx711.kicad_sch (KiCad schematic)
At the start: 13 parts, among them Q1 MMBT4403

Commit message: Further PCB tweaks
Connections:
- net HX_DAT renamed DAT
- net HX_GNDA renamed GNDA
- net HX_SCK renamed SCK
Changed lines of the file:
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@@
 (kicad_sch
-	(version 20231120)
+	(version 20250114)
 	(generator "eeschema")
-	(generator_version "8.0")
+	(generator_version "9.0")
 	(paper "A4")
+	(text "Analog/digital power and ground are tied together here.\nMaybe not ideal.\nhttps://github.com/sparkfun/HX711-Load-Cell-Amplifier/issues/7"
+		(exclude_from_sim no)
+		(at 101.092 163.576 0)
+		(effects
+			(font
+				(size 1.27 1.27)
+			)
+		)
+	)
 	(junction
 		(at 125.73 87.63)
@@
 		)
 	)
-	(text "Analog/digital power and ground are tied together here.\nMaybe not ideal.\nhttps://github.com/sparkfun/HX711-Load-Cell-Amplifier/issues/7"
-		(exclude_from_sim no)
-		(at 101.092 163.576 0)
+	(label "E+"
+		(at 64.77 87.63 0)
+		(effects
+			(font
+				(size 1.2446 1.2446)
+			)
+			(justify left bottom)
+		)
+	)
+	(label "A+"
+		(at 63.5 140.97 0)
+		(effects
+			(font
+				(size 1.2446 1.2446)
+			)
+			(justify left bottom)
+		)
+	)
+	(label "A-"
+		(at 64.77 128.27 0)
+		(effects
+			(font
+				(size 1.2446 1.2446)
+			)
+			(justify left bottom)
+		)
+	)
+	(label "SCK"
+		(at 189.23 109.22 0)
+		(effects
+			(font
+				(size 1.2446 1.2446)
+			)
+			(justify left bottom)
+		)
+	)
+	(label "DAT"
+		(at 189.23 106.68 0)
+		(effects
+			(font
+				(size 1.2446 1.2446)
+			)
+			(justify left bottom)
+		)
+	)
+	(hierarchical_label "GNDA"
+		(shape input)
+		(at 196.85 111.76 0)
 		(effects
 			(font
 				(size 1.27 1.27)
 			)
-		)
-	)
-	(label "E+"
-		(at 64.77 87.63 0)
-		(fields_autoplaced yes)
-		(effects
-			(font
-				(size 1.2446 1.2446)
-			)
-			(justify left bottom)
-		)
-	)
-	(label "A+"
-		(at 63.5 140.97 0)
-		(fields_autoplaced yes)
-		(effects
-			(font
-				(size 1.2446 1.2446)
-			)
-			(justify left bottom)
-		)
-	)
-	(label "A-"
-		(at 64.77 128.27 0)
-		(fields_autoplaced yes)
-		(effects
-			(font
-				(size 1.2446 1.2446)
-			)
-			(justify left bottom)
-		)
-	)
-	(label "SCK"
-		(at 189.23 109.22 0)
-		(fields_autoplaced yes)
-		(effects
-			(font
-				(size 1.2446 1.2446)
-			)
-			(justify left bottom)
-		)
-	)
-	(label "DAT"
-		(at 189.23 106.68 0)
-		(fields_autoplaced yes)
-		(effects
-			(font
-				(size 1.2446 1.2446)
-			)
-			(justify left bottom)
-		)
-	)
-	(hierarchical_label "HX_GNDA"
+			(justify left)
+		)
+	)
+	(hierarchical_label "DAT"
 		(shape input)
-		(at 196.85 111.76 0)
-		(fields_autoplaced yes)
+		(at 196.85 106.68 0)
 		(effects
 			(font
@@
 		)
 	)
-	(hierarchical_label "HX_DAT"
+	(hierarchical_label "SHLD"
 		(shape input)
-		(at 196.85 106.68 0)
-		(fields_autoplaced yes)
+		(at 60.96 147.32 180)
 		(effects
 			(font
 				(size 1.27 1.27)
 			)
-			(justify left)
-		)
-	)
-	(hierarchical_label "SHLD"
+			(justify right)
+		)
+	)
+	(hierarchical_label "E+"
 		(shape input)
-		(at 60.96 147.32 180)
-		(fields_autoplaced yes)
+		(at 60.96 87.63 180)
 		(effects
 			(font
@@
 		)
 	)
-	(hierarchical_label "E+"
+	(hierarchical_label "VDD"
 		(shape input)
-		(at 60.96 87.63 180)
-		(fields_autoplaced yes)
+		(at 196.85 101.6 0)
 		(effects
 			(font
 				(size 1.27 1.27)
 			)
-			(justify right)
-		)
-	)
-	(hierarchical_label "HX_VDD"
+			(justify left)
+		)
+	)
+	(hierarchical_label "A+"
 		(shape input)
-		(at 196.85 101.6 0)
-		(fields_autoplaced yes)
+		(at 60.96 140.97 180)
 		(effects
 			(font
 				(size 1.27 1.27)
 			)
-			(justify left)
-		)
-	)
-	(hierarchical_label "A+"
+			(justify right)
+		)
+	)
+	(hierarchical_label "A-"
 		(shape input)
-		(at 60.96 140.97 180)
-		(fields_autoplaced yes)
+		(at 60.96 128.27 180)
 		(effects
 			(font
@@
 		)
 	)
-	(hierarchical_label "A-"
+	(hierarchical_label "VCC"
 		(shape input)
-		(at 60.96 128.27 180)
-		(fields_autoplaced yes)
+		(at 196.85 99.06 0)
 		(effects
 			(font
 				(size 1.27 1.27)
 			)
-			(justify right)
-		)
-	)
-	(hierarchical_label "HX_VCC"
+			(justify left)
+		)
+	)
+	(hierarchical_label "E-"
 		(shape input)
-		(at 196.85 99.06 0)
-		(fields_autoplaced yes)
+		(at 60.96 118.11 180)
 		(effects
 			(font
 				(size 1.27 1.27)
 			)
-			(justify left)
-		)
-	)
-	(hierarchical_label "E-"
-		(shape input)
-		(at 60.96 118.11 180)
-		(fields_autoplaced yes)
-		(effects
-			(font
-				(size 1.27 1.27)
-			)
 			(justify right)
 		)
 	)
-	(hierarchical_label "HX_SCK"
+	(hierarchical_label "SCK"
 		(shape input)
 		(at 196.85 109.22 0)
-		(fields_autoplaced yes)
 		(effects
 			(font
@@
 			)
 		)
-		(property "Value" "HX_GNDA"
+		(property "Value" "GNDA"
 			(at 194.31 119.38 0)
 			(effects
@@
 			)
 		)
-		(property "Value" "HX_GNDA"
+		(property "Value" "GNDA"
 			(at 157.48 81.28 0)
 			(effects
@@
 			)
 		)
-		(property "Value" "HX_GNDA"
+		(property "Value" "GNDA"
 			(at 114.3 123.19 0)
 			(effects
@@
 			)
 		)
-		(property "Value" "HX_GNDA"
+		(property "Value" "GNDA"
 			(at 172.72 123.19 0)
 			(effects
@@
 			)
 		)
-		(property "Value" "HX_GNDA"
+		(property "Value" "GNDA"
 			(at 171.45 81.28 0)
 			(effects
@@
 			)
 		)
-		(property "Value" "HX_GNDA"
+		(property "Value" "GNDA"
 			(at 63.5 154.94 0)
 			(effects
